Commit message: 添加nav2与参数

File: description/lidar.xacro (robot description, xacro)
@@ -32,9 +32,9 @@
             <update_rate>10</update_rate>
             <topic>scan</topic>
-            <gz_frame_id>laser_frame</gz_frame_id>   <!-- ← 改这里，frame_id → gz_frame_id -->
+            <gz_frame_id>laser_frame</gz_frame_id>
             <lidar>
                 <scan>
                     <horizontal>
-                        <samples>360</samples>
+                        <samples>500</samples>
                         <min_angle>-3.14159</min_angle>
                         <max_angle>3.14159</max_angle>
@@ -42,6 +42,6 @@
                 </scan>
                 <range>
-                    <min>0.3</min>
-                    <max>12</max>
+                    <min>0.0699</min>
+                    <max>5.0001</max>
                 </range>
             </lidar>

File: description/robot_core.xacro (robot description, xacro)
@@ -24,5 +24,5 @@
         <parent link="base_footprint" />
         <child link="base_link" />
-        <origin xyz="0 0 0" rpy="0 0 0" />
+        <origin xyz="0 0 0.05" rpy="0 0 0" />
     </joint>
     <link name="base_footprint">
@@ -32,9 +32,9 @@
         <parent link="base_link" />
         <child link="chassis" />
-        <origin xyz="-0.1 0 0" />
+        <origin xyz="0 0 0" />
     </joint>
     <link name="chassis">
         <visual>
-            <origin xyz="0.15 0 0.075" rpy="0 0 0" />
+            <origin xyz="0.0 0 0.075" rpy="0 0 0" />
             <geometry>
                 <box size="0.3 0.3 0.15" />
@@ -43,14 +43,13 @@
         </visual>
         <collision>
-            <origin xyz="0.15 0.0 0.075" rpy="0.0 0.0 0.0" />
+            <origin xyz="0.0 0.0 0.075" rpy="0.0 0.0 0.0" />
             <geometry>
                 <box size="0.3 0.3 0.15" />
             </geometry>
         </collision>
-        <xacro:inertial_box mass="0.5" x="0.3" y="0.3" z="0.15">
-            <origin xyz="0.15 0 0.075" rpy="0 0 0" />
+        <xacro:inertial_box mass="3.5" x="0.3" y="0.3" z="0.15">
+            <origin xyz="0.0 0 0.075" rpy="0 0 0" />
         </xacro:inertial_box>
     </link>
-    <!-- 左轮 -->
     <joint name="left_wheel_joint" type="continuous">
         <parent link="base_link" />
@@ -58,5 +57,6 @@
         <origin xyz="0.0 0.175 0.0" rpy="-${pi/2} 0.0 0.0" />
         <axis xyz="0.0 0.0 1.0" />
-        <limit effort="0.05" velocity="10.0" />
+        <limit effort="100.0" velocity="10.0" />
+        <dynamics damping="0.2" friction="0.2" />
     </joint>
     <link name="left_wheel">
@@ -68,14 +68,22 @@
         </visual>
         <collision>
-            <!-- 碰撞检测改为圆形，减少摩檫力 -->
             <geometry>
                 <sphere radius="0.05" />
             </geometry>
         </collision>
-        <xacro:inertial_cylinder mass="0.1" length="0.04" radius="0.05">
+        <xacro:inertial_cylinder mass="0.25" length="0.04" radius="0.05">
             <origin xyz="0 0 0" rpy="0 0 0" />
         </xacro:inertial_cylinder>
     </link>
-    <!-- 右轮 -->
+    <gazebo reference="left_wheel">
+        <mu1>1.0</mu1>
+        <mu2>0.5</mu2>
+        <kp>500000.0</kp>
+        <kd>10.0</kd>
+        <minDepth>0.001</minDepth>
+        <maxVel>0.1</maxVel>
+        <fdir1>1 0 0</fdir1>
+        <material>Gazebo/Blue</material>
+    </gazebo>
     <joint name="right_wheel_joint" type="continuous">
         <parent link="base_link" />
@@ -83,5 +91,6 @@
         <origin xyz="0.0 -0.175 0.0" rpy="${pi/2} 0.0 0.0" />
         <axis xyz="0.0 0.0 -1.0" />
-        <limit effort="0.05" velocity="10.0" />
+        <limit effort="100.0" velocity="10.0" />
+        <dynamics damping="0.2" friction="0.2" />
     </joint>
     <link name="right_wheel">
@@ -94,19 +103,28 @@
         <collision>
             <geometry>
-                <!-- 碰撞检测改为圆形，减少摩檫力 -->
                 <sphere radius="0.05" />
             </geometry>
         </collision>
-        <xacro:inertial_cylinder mass="0.1" length="0.04" radius="0.05">
+        <xacro:inertial_cylinder mass="0.25" length="0.04" radius="0.05">
             <origin xyz="0 0 0" rpy="0 0 0" />
         </xacro:inertial_cylinder>
     </link>
-    <!-- 万向辅助轮 -->
-    <joint name="caster_wheel_joint" type="fixed">
+    <gazebo reference="right_wheel">
+        <mu1>100000.0</mu1>
+        <mu2>100000.0</mu2>
+        <kp>1000000.0</kp>
+        <kd>100.0</kd>
+        <minDepth>0.001</minDepth>
+        <maxVel>0.1</maxVel>
+        <fdir1>1 0 0</fdir1>
+        <material>Gazebo/Blue</material>
+    </gazebo>
+    <!-- 前辅助轮 -->
+    <joint name="caster_front_joint" type="fixed">
         <parent link="chassis" />
-        <child link="caster_wheel" />
-        <origin xyz="0.24 0 0" rpy="0 0 0" />
+        <child link="caster_front_wheel" />
+        <origin xyz="0.12 0 0" rpy="0 0 0" />
     </joint>
-    <link name="caster_wheel">
+    <link name="caster_front_wheel">
         <visual>
             <geometry>
@@ -124,7 +142,43 @@
         </xacro:inertial_sphere>
     </link>
-    <gazebo reference="caster_wheel">
-        <mu1 value="0.0001" />
-        <mu1 value="0.0001" />
+    <gazebo reference="caster_front_wheel">
+        <mu1>0.0001</mu1>
+        <mu2>0.0001</mu2>
+        <kp>1000000.0</kp>
+        <kd>100.0</kd>
+        <minDepth>0.001</minDepth>
+        <maxVel>1.0</maxVel>
+        <material>Gazebo/Black</material>
+    </gazebo>
+    <!-- 后辅助轮 -->
+    <joint name="caster_back_joint" type="fixed">
+        <parent link="chassis" />
+        <child link="caster_back_wheel" />
+        <origin xyz="-0.12 0 0" rpy="0 0 0" />   <!-- 后方对称位置 -->
+    </joint>
+    <link name="caster_back_wheel">
+        <visual>
+            <geometry>
+                <sphere radius="0.05" />
+            </geometry>
+            <material name="black" />
+        </visual>
+        <collision>
+            <geometry>
+                <sphere radius="0.05" />
+            </geometry>
+        </collision>
+        <xacro:inertial_sphere mass="0.1" radius="0.05">
+            <origin xyz="0 0 0" rpy="0 0 0" />
+        </xacro:inertial_sphere>
+    </link>
+    <gazebo reference="caster_back_wheel">
+        <mu1>0.0001</mu1>
+        <mu2>0.0001</mu2>
+        <kp>1000000.0</kp>
+        <kd>100.0</kd>
+        <minDepth>0.001</minDepth>
+        <maxVel>1.0</maxVel>
+        <material>Gazebo/Black</material>
     </gazebo>
 </robot>
